File: hardware/YAKB.kicad_pcb (KiCad board)
At the start: 4 copper layers, 285 x 94.6 mm, 103 parts, among them J1 Battery_PH2.0, Q1 AO3401A, SW1 Battery_switch_pigtail, SW2 Reset_NO, U1 nice!nano_v2, U2 SN74HC4051D, U3 SN74HC4051D, U4 OPA350UA

Commit message: fix: validate YAKB hardware, hide fasteners and add battery options
Parts:
- J1: value Battery_PH2.0 -> JST_S2B-PH-K
- U2, U3: value SN74HC4051D -> CD74HC4051M96
- moved C3 12.4 mm to (220.0, 88.0)
- moved U4 6.00 mm to (217.0, 84.0)
- turned U1 to 0 degrees
Routing:
- net GND: track 2569.1 -> 2458.2 mm, vias 67 -> 79
- net DRAIN: track 16.6 -> 47.2 mm
- net MUX0_INH: track 160.3 -> 189.4 mm, vias 1 -> 2
- net MUX_C: track 155.1 -> 181.3 mm
- net RESET: track 35.3 -> 14.2 mm, vias 1 -> 0
- net ROW_DRV1: track 234.8 -> 215.9 mm
- net AFE_ON_N: track 47.0 -> 65.6 mm, vias 1 -> 2
- net AFE_3V3: track 42.0 -> 25.2 mm, vias 2 -> 0
- net ROW_DRV0: track 237.4 -> 220.9 mm, vias 0 -> 1
- net ROW_DRV2: track 219.7 -> 205.8 mm
- net ADC: track 46.9 -> 58.7 mm
- net ROW_DRV3: track 220.8 -> 213.4 mm, vias 1 -> 2
- net VCC: track 245.1 -> 238.0 mm
- net FB: track 27.1 -> 21.0 mm
- net MUX_B: track 194.2 -> 199.4 mm, vias 6 -> 5
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