File: hardware/YAKB.kicad_sch (KiCad schematic)
At the start: 100 parts, among them J1 Battery_PH2.0, Q1 AO3401A, SW1 Battery_switch_pigtail, SW2 Reset_NO, U1 nice!nano_v2, U2 SN74HC4051D, U3 SN74HC4051D, U4 OPA350UA

Commit message: fix: validate YAKB hardware, hide fasteners and add battery options
Parts:
- J1: value Battery_PH2.0 -> JST_S2B-PH-K
- U2, U3: value SN74HC4051D -> CD74HC4051M96
