File: hardware/modular/YAKB-shaped-FPC-B1.kicad_sch (KiCad schematic)
At the start: 2 parts

Commit message: fix(hardware): correct FPC mating geometry and add fit coupons
Parts:
- J_A, J_B: value FPC_BOTTOM_CONTACT_1mm -> MOLEX_200528_1mm_BOTTOM
